File: hardware/adc.kicad_sch (KiCad schematic)
At the start: 29 parts, among them J6 ANALOG_SEL, U4 MCP3204, U9 PJ-320A

Commit message: feat(hw): closing sch, starting pcb
Parts:
- removed D22, D23: BAT54J, Package_TO_SOT_SMD:SOT-323_SC-70, symbol Diode:BAT54J
- added D8: BAV199DW, Package_TO_SOT_SMD:SOT-363_SC-70-6, symbol Diode:BAV199DW
- renumbered C17 to C14, C34 to C15, C35 to C16, C36 to C17, C33 to C18, J6 to J5, R98 to R76, R99 to R77, R89 to R78, R88 to R79, R90 to R80, R91 to R81, R96 to R82, R87 to R83, R97 to R84, R92 to R85, TP41 to TP22, TP40 to TP23, TP6 to TP24, TP4 to TP25, TP42 to TP26, TP45 to TP27, TP44 to TP28, TP43 to TP29, U9 to U6, U4 to U7
Connections:
- net +3V3_ANA: now also D8.2 (K2)
- net at R83.2, R84.1: now also D8.6 (K3A4)
