File: hardware/dac.kicad_sch (KiCad schematic)
At the start: 29 parts, among them U8 MCP6001-OT

Commit message: feat(hw): closing sch, starting pcb
Parts:
- removed R70, R71, R73, R74, R75, R76, R77, R78, R85: 20k0.1%, Resistor_SMD:R_0603_1608Metric, symbol Device:R
- added C22: 0.1u, Capacitor_SMD:C_0603_1608Metric_Pad1.08x0.95mm_HandSolder, symbol Device:C
- added FB3: BLM18HE152SN1D, Inductor_SMD:L_0603_1608Metric, symbol Device:FerriteBead
- added R100, R102, R103, R105, R106, R108, R109, R110, R111, R87, R88, R90, R91, R93, R94, R96, R97, R99: 10k1%, Resistor_SMD:R_0603_1608Metric, symbol Device:R
- R101: renamed from R82; value 10k0.1% -> 10k1%
- R104: renamed from R83; value 10k0.1% -> 10k1%
- R107: renamed from R84; value 10k0.1% -> 10k1%
- R89: renamed from R72; value 10k0.1% -> 10k1%
- R92: renamed from R79; value 10k0.1% -> 10k1%
- R95: renamed from R80; value 10k0.1% -> 10k1%
- R98: renamed from R81; value 10k0.1% -> 10k1%
- renumbered C22 to C19, C18 to C20, C16 to C21, C21 to C23, R93 to R112, TP47 to TP30, TP48 to TP31, TP8 to TP32, TP7 to TP33, TP46 to TP34
Connections:
- net +3V3: now also FB3.2; no longer 595_5.16 (VCC)
- net GND: now also C22.2, R111.2
- net at R107.2: now also R109.1, R110.1
- net at C20.1, C21.1, R89.1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: now also R88.1
- net at 595_5.15 (QA): now also R87.1
- net at R95.2, R98.1: now also R97.1
- net at R101.1, R98.2: now also R100.1
- net at R89.2, R92.1: now also R91.1
- net at 595_5.1 (QB): now also R90.1
- net at 595_5.7 (QH): now also R108.1
- net at 595_5.3 (QD): now also R96.1
- net at R92.2, R95.1: now also R94.1
- net at 595_5.2 (QC): now also R93.1
- net at 595_5.4 (QE): now also R99.1
- net at 595_5.5 (QF): now also R102.1
- net at 595_5.6 (QG): now also R105.1
- net at R104.2, R107.1: now also R106.1
- net at R101.2, R104.1: now also R103.1
- new net: R108.2, R109.2
- new net: R105.2, R106.2
- new net: R100.2, R99.2
- new net: 595_5.16 (VCC), C22.1, FB3.1
- new net: R90.2, R91.2
- new net: R102.2, R103.2
- new net: R93.2, R94.2
- new net: R87.2, R88.2
- new net: R110.2, R111.1
- new net: R96.2, R97.2
Other:
- moved on the sheet: C23
