File: hardware/gatebench.kicad_pcb (KiCad board)
At the start: 2 copper layers, 286 parts, among them J1 Conn_01x02_Pin, J2 Screw_Terminal_01x02, J3 USB_B, J4 DE15_Socket_HighDensity_Mount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, J5 Conn_01x02_Pin, J6 ANALOG_SEL, J7 PMOD, J9 Qwiic | STEMMA QT, Q2 MMBT3906, Q3 MMBT3906, Q4 MMBT3906, Q5 MMBT3906, SW1 SW_SPDT, SW10 SW_SPDT, SW11 SW_SPDT, SW12 SW_SPDT, SW13 SW_SPDT, SW14 SW_SPDT, SW15 SW_SPDT, SW16 SW_SPDT, SW17 RotaryEncoder, SW18 SW_DIP_x02, SW2 SW_SPDT, SW3 SW_SPDT, SW4 SW_SPDT, SW5 SW_SPDT, SW6 SW_SPDT, SW7 SW_SPDT, SW8 SW_SPDT, SW9 SW_SPDT, U1 CA56-12EWA, U2 CH340N, U3 24LC02, U4 MCP3204, U5 AP2112K-3.3, U6 74AHCT1G125, U7 UPduinoV3_1Board, U8 MCP6001-OT, U9 PJ-320A

Commit message: feat(hw): closing sch, starting pcb
Parts:
- removed BTN0: SW_Push, Button_Switch_THT:SW_PUSH_6mm_H8.5mm
- removed D22, D23: BAT54J, Package_TO_SOT_SMD:SOT-323_SC-70
- removed D24, D25: RED, LED_SMD:LED_0603_1608Metric
- removed J9: Qwiic | STEMMA QT, footprints:CONN_SM04B_JST
- removed JP2: SolderJumper_3_Bridged12, Jumper:SolderJumper-3_P1.3mm_Bridged2Bar12_RoundedPad1.0x1.5mm_NumberLabels
- removed LED0: GREEN, LED_SMD:LED_0603_1608Metric
- removed Q5: MMBT3906, Button_Switch_SMD:Nidec_Copal_CAS-120A
- removed TP44, TP45, TP46, TP47, TP48, TP49, TP50, TP51, TP52, TP53, TP54: TestPoint_Alt, Connector_PinHeader_2.54mm:PinHeader_1x01_P2.54mm_Vertical
- added BTN1: SW_Push, Button_Switch_THT:SW_PUSH_6mm_H8.5mm, F.Cu at (373.6, 75.2)
- added C37: 10u, Capacitor_SMD:C_0603_1608Metric_Pad1.08x0.95mm_HandSolder, F.Cu at (464.3, 161.2)
- added C38: 10u, Capacitor_SMD:C_0603_1608Metric_Pad1.08x0.95mm_HandSolder, F.Cu at (464.3, 163.7)
- added C39: 0.1u, Capacitor_SMD:C_0603_1608Metric_Pad1.08x0.95mm_HandSolder, F.Cu at (464.3, 166.2)
- added C4: 1nF/250V, Capacitor_SMD:C_0603_1608Metric_Pad1.08x0.95mm_HandSolder, F.Cu at (111.1, 32.4)
- added C40: 0.1u, Capacitor_SMD:C_0603_1608Metric_Pad1.08x0.95mm_HandSolder, F.Cu at (464.3, 168.7)
- added D15: WS2812B, LED_SMD:LED_WS2812B_PLCC4_5.0x5.0mm_P3.2mm, F.Cu at (361.3, 153.4)
- added D16: WS2812B, LED_SMD:LED_WS2812B_PLCC4_5.0x5.0mm_P3.2mm, F.Cu at (361.3, 160.0)
- added D17: WS2812B, LED_SMD:LED_WS2812B_PLCC4_5.0x5.0mm_P3.2mm, F.Cu at (361.3, 166.6)
- added D18: WS2812B, LED_SMD:LED_WS2812B_PLCC4_5.0x5.0mm_P3.2mm, F.Cu at (361.3, 173.3)
- added FB3: BLM18HE152SN1D, Inductor_SMD:L_0603_1608Metric, F.Cu at (453.3, 76.8)
- added H1: MountingHole, MountingHole:MountingHole_3.2mm_M3, F.Cu at (77.9, 26.7)
- added H2: MountingHole, MountingHole:MountingHole_3.2mm_M3, F.Cu at (216.6, 27.4)
- added H3: MountingHole, MountingHole:MountingHole_3.2mm_M3, F.Cu at (78.4, 165.3)
- added H4: MountingHole, MountingHole:MountingHole_3.2mm_M3, F.Cu at (215.8, 165.0)
- added J8: PMOD, Connector_PinHeader_2.54mm:PinHeader_2x06_P2.54mm_Horizontal, F.Cu at (447.5, 148.4)
- added JP3: Jumper_2_Open, TestPoint:TestPoint_2Pads_Pitch2.54mm_Drill0.8mm, F.Cu at (251.4, 58.6)
- added LED16: YELLOW, LED_SMD:LED_0603_1608Metric, F.Cu at (436.6, 112.5)
- added Q1: MMBT3906, Button_Switch_SMD:Nidec_Copal_CAS-120A, F.Cu at (413.1, 141.2)
- added R100: 10k1%, Resistor_SMD:R_0603_1608Metric, F.Cu at (457.4, 94.3)
- added R101: 10k1%, Resistor_SMD:R_0603_1608Metric, F.Cu at (461.4, 76.8)
- added R102: 10k1%, Resistor_SMD:R_0603_1608Metric, F.Cu at (461.4, 79.3)
- added R103: 10k1%, Resistor_SMD:R_0603_1608Metric, F.Cu at (461.4, 81.8)
- added R104: 10k1%, Resistor_SMD:R_0603_1608Metric, F.Cu at (461.4, 84.3)
- added R105: 10k1%, Resistor_SMD:R_0603_1608Metric, F.Cu at (461.4, 86.8)
- added R106: 10k1%, Resistor_SMD:R_0603_1608Metric, F.Cu at (461.4, 89.3)
- added R107: 10k1%, Resistor_SMD:R_0603_1608Metric, F.Cu at (461.4, 91.8)
- added R108: 10k1%, Resistor_SMD:R_0603_1608Metric, F.Cu at (461.4, 94.3)
- added TP1: TestPoint_Alt, Connector_PinHeader_2.54mm:PinHeader_1x01_P2.54mm_Vertical, F.Cu at (373.8, 44.5)
- added TP10: TestPoint_Alt, Connector_PinHeader_2.54mm:PinHeader_1x01_P2.54mm_Vertical, F.Cu at (90.4, 54.4)
- added TP11: TestPoint_Alt, Connector_PinHeader_2.54mm:PinHeader_1x01_P2.54mm_Vertical, F.Cu at (275.0, 42.4)
- added TP12: TestPoint_Alt, Connector_PinHeader_2.54mm:PinHeader_1x01_P2.54mm_Vertical, F.Cu at (275.0, 37.8)
- added TP13: TestPoint_Alt, Connector_PinHeader_2.54mm:PinHeader_1x01_P2.54mm_Vertical, F.Cu at (275.0, 33.2)
- added TP16: TestPoint_Alt, Connector_PinHeader_2.54mm:PinHeader_1x01_P2.54mm_Vertical, F.Cu at (270.4, 42.4)
- added TP17: TestPoint_Alt, Connector_PinHeader_2.54mm:PinHeader_1x01_P2.54mm_Vertical, F.Cu at (270.4, 37.8)
- added TP18: TestPoint_Probe, TestPoint:TestPoint_Loop_D2.60mm_Drill0.9mm_Beaded, F.Cu at (253.3, 36.6)
- added TP19: TestPoint_Alt, Connector_PinHeader_2.54mm:PinHeader_1x01_P2.54mm_Vertical, F.Cu at (270.4, 33.2)
- added TP20: TestPoint_Probe, TestPoint:TestPoint_Loop_D2.60mm_Drill0.9mm_Beaded, F.Cu at (253.3, 31.6)
- added TP21: TestPoint_Alt, Connector_PinHeader_2.54mm:PinHeader_1x01_P2.54mm_Vertical, F.Cu at (270.4, 28.6)
- added TP22: TestPoint_Alt, Connector_PinHeader_2.54mm:PinHeader_1x01_P2.54mm_Vertical, F.Cu at (457.6, 66.6)
- added TP5: TestPoint_Alt, Connector_PinHeader_2.54mm:PinHeader_1x01_P2.54mm_Vertical, F.Cu at (378.4, 44.5)
- added TP9: TestPoint_Probe, TestPoint:TestPoint_Loop_D2.60mm_Drill0.9mm_Beaded, F.Cu at (80.7, 45.8)
- added U10: SRV05-4, Package_TO_SOT_SMD:SOT-23-5, F.Cu at (464.7, 148.4)
- added U11: SRV05-4, Package_TO_SOT_SMD:SOT-23-5, F.Cu at (464.7, 153.1)
- added U12: SRV05-4, Package_TO_SOT_SMD:SOT-23-5, F.Cu at (464.7, 157.7)
- C1, C2: value 10n -> 0.1u
- C12, C13: value 0.1u -> 10n
- C14, C26, C7: value 0.1u -> 10u
- C15: value 0.1u -> 1u
- C16: value 47p -> 33n
- C17: value 10u -> 22n
- C18: value 0805 -> 1u
- C19, C32, C8: value 10u -> 0.1u
- C20: value 0.1u -> 0805
- C21: value 0.1u -> 47p
- C24: value 0.1u -> 1nF/250V
- C3: value 1nF/250V -> 0.1u
- C33: value 1u -> 0.1u
- C35: value 33n -> 0.1u
- C36: value 22n -> 0.1u
- C5: value 1nF/250V -> 10u
- D1: value PMEG2010EH -> BAV199DW; footprint Package_TO_SOT_SMD:SOT-583-8 -> Package_TO_SOT_SMD:SOT-363_SC-70-6
- D2: value SMF5V0A -> PMEG2010EH; footprint Diode_SMD:D_SMF -> Package_TO_SOT_SMD:SOT-583-8
- D3: footprint Package_TO_SOT_SMD:SOT-583-8 -> Diode_SMD:Nexperia_CFP3_SOD-123W
- D4: value BAT54J -> SMF5V0A; footprint Package_TO_SOT_SMD:SOT-323_SC-70 -> Diode_SMD:D_SMF
- D5: value WS2812B -> BAT54J; footprint LED_SMD:LED_WS2812B_PLCC4_5.0x5.0mm_P3.2mm -> Package_TO_SOT_SMD:SOT-323_SC-70
- D6, D7: value WS2812B -> RED; footprint LED_SMD:LED_WS2812B_PLCC4_5.0x5.0mm_P3.2mm -> LED_SMD:LED_0603_1608Metric
- D8: value WS2812B -> BAV199DW; footprint LED_SMD:LED_WS2812B_PLCC4_5.0x5.0mm_P3.2mm -> Package_TO_SOT_SMD:SOT-363_SC-70-6
- J4: value DE15_Socket_HighDensity_MountingHoles -> Conn_01x02_Pin; footprint Connector_Dsub:DSUB-15-HD_Socket_Horizontal_P2.29x2.54mm_EdgePinOffset8.35mm_Housed_MountingHolesOffset10.89mm -> Connector_PinHeader_2.54mm:PinHeader_1x02_P2.54mm_Vertical
- J5: value Conn_01x02_Pin -> ANALOG_SEL; footprint Connector_PinHeader_2.54mm:PinHeader_1x02_P2.54mm_Vertical -> Connector_PinHeader_2.54mm:PinHeader_1x03_P2.54mm_Vertical
- J6: value ANALOG_SEL -> DE15_Socket_HighDensity_MountingHoles; footprint Connector_PinHeader_2.54mm:PinHeader_1x03_P2.54mm_Vertical -> Connector_Dsub:DSUB-15-HD_Socket_Horizontal_P2.29x2.54mm_EdgePinOffset8.35mm_Housed_MountingHolesOffset10.89mm
- J7: value PMOD -> Qwiic | STEMMA QT; footprint Connector_PinHeader_2.54mm:PinHeader_2x06_P2.54mm_Horizontal -> footprints:CONN_SM04B_JST
- JP1: value Jumper_2_Open -> SolderJumper_3_Bridged12; footprint TestPoint:TestPoint_2Pads_Pitch2.54mm_Drill0.8mm -> Jumper:SolderJumper-3_P1.3mm_Bridged2Bar12_RoundedPad1.0x1.5mm_NumberLabels
- LED8: value YELLOW -> GREEN
- R1, R2: value 10k -> 4k7
- R10, R13, R16: value 2k1% -> 100
- R109, R110, R111: value 100 -> 10k1%
- R11, R14, R17: value 1k1% -> 100
- R112: value 100 -> 10k
- R113, R116, R119: value 100 -> 2k1%
- R114, R117, R120: value 100 -> 1k1%
- R115, R118, R121: value 100 -> 510-1%
- R12, R15, R18: value 510-1% -> 100
- R122: value 100 -> 1M
- R125: value 100 -> 330
- R19, R20, R3, R4, R5, R7, R9: value 10k -> 100
- R21: value 10k -> 1M
- R22: value 1M -> 4k7
- R23: value 100 -> 4k7
- R24: value 100 -> 1k
- R25: value 4k7 -> 470
- R26, R27, R28: value 4k7 -> 10k
- R29, R38, R39, R40, R41, R42, R43: value 330 -> 10k
- R44, R45: value 330 -> 220
- R46, R47: value 470 -> 220
- R48, R49, R50, R51, R52, R53, R54, R55: value 470 -> 330
- R56, R57, R58, R59: value 470 -> 2k2
- R62, R63, R64, R65: value 2k2 -> 470
- R66, R67, R68, R69: value 220 -> 470
- R70, R71, R73, R74, R75: value 20k0.1% -> 470
- R72: value 10k0.1% -> 470
- R76, R77: value 20k0.1% -> 1k
- R78, R85: value 20k0.1% -> 10k
- R79, R81, R82: value 10k0.1% -> 10k
- R8: value 1M -> 100
- R80: value 10k0.1% -> R_Photo; footprint Resistor_SMD:R_0603_1608Metric -> OptoDevice:R_LDR_7x6mm_P5.1mm_Vertical
- R83: value 10k0.1% -> 1k
- R84: value 10k0.1% -> 330
- R87, R94, R96, R98, R99: value 1k -> 10k1%
- R88, R89, R91, R92, R93: value 10k -> 10k1%
- R90: value R_Photo -> 10k1%; footprint OptoDevice:R_LDR_7x6mm_P5.1mm_Vertical -> Resistor_SMD:R_0603_1608Metric
- R95: value 470 -> 10k1%
- R97: value 330 -> 10k1%
- SW17: value RotaryEncoder -> SW_DIP_x02; footprint Rotary_Encoder:RotaryEncoder_Alps_EC11E-Switch_Vertical_H20mm -> Button_Switch_THT:SW_DIP_SPSTx02_Slide_9.78x7.26mm_W7.62mm_P2.54mm
- SW18: value SW_DIP_x02 -> RotaryEncoder; footprint Button_Switch_THT:SW_DIP_SPSTx02_Slide_9.78x7.26mm_W7.62mm_P2.54mm -> Rotary_Encoder:RotaryEncoder_Alps_EC11E-Switch_Vertical_H20mm
- TP14, TP15, TP2, TP3, TP4, TP6, TP7: value TestPoint_Probe -> TestPoint_Alt; footprint TestPoint:TestPoint_Loop_D2.60mm_Drill0.9mm_Beaded -> Connector_PinHeader_2.54mm:PinHeader_1x01_P2.54mm_Vertical
- TP24, TP25, TP32, TP33: value TestPoint_Alt -> TestPoint_Probe; footprint Connector_PinHeader_2.54mm:PinHeader_1x01_P2.54mm_Vertical -> TestPoint:TestPoint_Loop_D2.60mm_Drill0.9mm_Beaded
- U1: value CA56-12EWA -> 24LC02; footprint Display_7Segment:CA56-12EWA -> Package_SO:SOIC-8_3.9x4.9mm_P1.27mm
- U2: value CH340N -> UPduinoV3_1Board; footprint Package_SO:JEITA_SOIC-8_3.9x4.9mm_P1.27mm -> upduino_v3_1:upduino_v3_1
- U3: value 24LC02 -> AP2112K-3.3; footprint Package_SO:SOIC-8_3.9x4.9mm_P1.27mm -> Package_TO_SOT_SMD:SOT-23-5
- U4: value MCP3204 -> CH340N; footprint Package_SO:SOIC-14_3.9x8.7mm_P1.27mm -> Package_SO:JEITA_SOIC-8_3.9x4.9mm_P1.27mm
- U5: value AP2112K-3.3 -> CA56-12EWA; footprint Package_TO_SOT_SMD:SOT-23-5 -> Display_7Segment:CA56-12EWA
- U6: value 74AHCT1G125 -> PJ-320A; footprint Package_TO_SOT_SMD:SOT-23-5 -> PJ-320A_Library:PJ-320A
- U7: value UPduinoV3_1Board -> MCP3204; footprint upduino_v3_1:upduino_v3_1 -> Package_SO:SOIC-14_3.9x8.7mm_P1.27mm
- U9: value PJ-320A -> 74AHCT1G125; footprint PJ-320A_Library:PJ-320A -> Package_TO_SOT_SMD:SOT-23-5
- moved C17 424.9 mm to (473.0, 58.8)
- moved R90 416.7 mm to (453.3, 89.3)
- moved RV1 416.7 mm to (457.0, 54.6)
- moved C19 415.6 mm to (474.1, 76.8)
- moved C20 415.6 mm to (474.1, 79.3)
- moved R91 402.5 mm to (453.3, 91.8)
- moved R92 402.5 mm to (453.3, 94.3)
- moved R87 402.5 mm to (453.3, 81.8)
- moved R88 402.5 mm to (453.3, 84.3)
- moved R89 402.5 mm to (453.3, 86.8)
- moved C23 400.9 mm to (474.1, 86.8)
- moved C15 400.7 mm to (473.0, 53.7)
- moved D8 396.0 mm to (453.3, 66.7)
- moved U6 385.3 mm to (456.1, 43.9)
- moved R80 383.8 mm to (473.7, 46.0)
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Connections:
- 165_1 pad 10: /Input Chain/165_2_TO_1 -> /Input Chain/165_4_TO_3
- 165_1 pad 11: Net-(165_1-D0) -> /Input Chain/SW0
- 165_1 pad 12: Net-(165_1-D1) -> /Input Chain/SW1
- 165_1 pad 13: /Input Chain/SEL_0 -> /Input Chain/SW2
- 165_1 pad 14: /Input Chain/SEL_1 -> /Input Chain/SW3
- 165_1 pad 3: /Input Chain/ENC_SW -> /Input Chain/SW4
- 165_1 pad 4: /Input Chain/ENC_B -> /Input Chain/SW5
- 165_1 pad 5: /Input Chain/ENC_A -> /Input Chain/SW6
- 165_1 pad 6: /Input Chain/KB_ROW1 -> /Input Chain/SW7
- 165_1 pad 9: SIN_DOUT -> /Input Chain/165_3_TO_2
- 165_2 pad 10: /Input Chain/165_3_TO_2 -> GND
- 165_2 pad 11: /Input Chain/KB_ROW2 -> /Input Chain/SW8
- 165_2 pad 12: /Input Chain/KB_ROW3 -> /Input Chain/SW9
- 165_2 pad 13: /Input Chain/KB_ROW4 -> /Input Chain/SW10
- 165_2 pad 14: /Input Chain/BTN_CENTER -> /Input Chain/SW11
- 165_2 pad 3: /Input Chain/BTN_RIGHT -> /Input Chain/SW12
- 165_2 pad 4: /Input Chain/BTN_LEFT -> /Input Chain/SW13
- 165_2 pad 5: /Input Chain/BTN_DOWN -> /Input Chain/SW14
- 165_2 pad 6: /Input Chain/BTN_UP -> /Input Chain/SW15
- 165_2 pad 9: /Input Chain/165_2_TO_1 -> /Input Chain/165_4_TO_3
- 165_3 pad 10: /Input Chain/165_4_TO_3 -> /Input Chain/165_3_TO_2
- 165_3 pad 11: /Input Chain/SW0 -> /Input Chain/KB_ROW2
- 165_3 pad 12: /Input Chain/SW1 -> /Input Chain/KB_ROW3
- 165_3 pad 13: /Input Chain/SW2 -> /Input Chain/KB_ROW4
- 165_3 pad 14: /Input Chain/SW3 -> /Input Chain/BTN_CENTER
- 165_3 pad 3: /Input Chain/SW4 -> /Input Chain/BTN_RIGHT
- 165_3 pad 4: /Input Chain/SW5 -> /Input Chain/BTN_LEFT
- 165_3 pad 5: /Input Chain/SW6 -> /Input Chain/BTN_DOWN
- 165_3 pad 6: /Input Chain/SW7 -> /Input Chain/BTN_UP
- 165_3 pad 9: /Input Chain/165_3_TO_2 -> /Input Chain/165_2_TO_1
- 165_4 pad 10: GND -> /Input Chain/165_2_TO_1
- 165_4 pad 11: /Input Chain/SW8 -> Net-(165_4-D0)
- 165_4 pad 12: /Input Chain/SW9 -> Net-(165_4-D1)
- 165_4 pad 13: /Input Chain/SW10 -> /Input Chain/SEL_0
- 165_4 pad 14: /Input Chain/SW11 -> /Input Chain/SEL_1
- 165_4 pad 3: /Input Chain/SW12 -> /Input Chain/ENC_SW
- 165_4 pad 4: /Input Chain/SW13 -> /Input Chain/ENC_B
- 165_4 pad 5: /Input Chain/SW14 -> /Input Chain/ENC_A
- 165_4 pad 6: /Input Chain/SW15 -> /Input Chain/KB_ROW1
- 165_4 pad 9: /Input Chain/165_4_TO_3 -> SIN_DOUT
- 595_5 pad 11: SPI_SCK -> PMOD_9
- 595_5 pad 14: SPI_MOSI -> PMOD_8
- 595_5 pad 16: +3V3 -> Net-(595_5-VCC)
- C1 pad 1: /Input Chain/ENC_A -> +3V3
- C10 pad 1: +3V3 -> +3V3_ANA
- C11 pad 1: +3V3 -> +3V3_ANA
- C12 pad 1: +5V -> /Input Chain/ENC_A
- C13 pad 1: +5V_UP -> /Input Chain/ENC_B
- C14 pad 1: +3V3_UP -> Net-(J5-Pin_3)
- C14 pad 2: GND -> /ADC/AUDIO_IN
- C15 pad 1: GND -> /ADC/ADC_CH0
- C15 pad 2: +5V -> GND
- C16 pad 1: Net-(U8-+) -> /ADC/ADC_CH2
- C17 pad 1: Net-(J6-Pin_3) -> /ADC/ADC_CH1
- C17 pad 2: /ADC/AUDIO_IN -> GND
- C18 pad 1: Net-(U8-+) -> +3V3_ANA
- C2 pad 1: /Input Chain/ENC_B -> +5V_UP
- C20 pad 1: +3V3_ANA -> Net-(U8-+)
- C21 pad 1: +3V3 -> Net-(U8-+)
- C22 pad 1: +3V3_ANA -> Net-(595_5-VCC)
- C23 pad 1: GND -> +3V3
- C23 pad 2: +5V -> GND
- C24 pad 2: +5V -> Net-(C24-Pad2)
- C25 pad 1: GND -> +5V
- C25 pad 2: +5V -> GND
- C26 pad 1: GND -> +5V
- C26 pad 2: +5V -> GND
- C3 pad 1: GND -> +3V3_UP
- C3 pad 2: Net-(J3-Shield) -> GND
- C32 pad 1: +5V -> GND
- C32 pad 2: GND -> +5V
- C33 pad 1: +3V3_ANA -> GND
- C33 pad 2: GND -> +5V
- C34 pad 1: /ADC/ADC_CH0 -> GND
- C34 pad 2: GND -> +5V
- C35 pad 1: /ADC/ADC_CH2 -> GND
- C35 pad 2: GND -> +5V
- C36 pad 1: /ADC/ADC_CH1 -> GND
- C36 pad 2: GND -> +5V
- C5 pad 1: GND -> +5V
- C5 pad 2: Net-(C5-Pad2) -> GND
- C6 pad 1: +3V3 -> +5V
- C8 pad 1: +5V -> +3V3
- C9 pad 1: +5V -> +3V3
- D1 pad 1: VBUS -> GND
- D1 pad 2: Net-(D1-A) -> +3V3
- D1 pad 6: (no net) -> /CLK_12M_EXT
- D11 pad 4: Net-(D10-DOUT) -> Net-(D11-DIN)
- D12 pad 2: Net-(D12-DOUT) -> Net-(D10-DIN)
- D12 pad 4: Net-(D11-DOUT) -> Net-(D12-DIN)
- D13 pad 4: Net-(D12-DOUT) -> Net-(D11-DOUT)
- D14 pad 2: Net-(D14-DOUT) -> Net-(D12-DIN)
- D14 pad 4: Net-(D13-DOUT) -> Net-(D14-DIN)
- D2 pad 1: Net-(D2-A1) -> Net-(D2-K)
- D2 pad 2: GND -> +5V
- D3 pad 1: Net-(D3-K) -> VBUS
- D3 pad 2: +5V -> /Power & USB/preVBUS
- D4 pad 1: Net-(D4-K) -> Net-(D4-A1)
- D4 pad 2: RX -> GND
- D5 pad 1: +5V -> Net-(D5-K)
- D5 pad 2: Net-(D5-DOUT) -> UART_RX
- D5 pad 3: GND -> (no net)
- D6 pad 1: +5V -> GND
- D6 pad 2: Net-(D6-DOUT) -> Net-(D6-A)
- D7 pad 1: +5V -> GND
- D7 pad 2: Net-(D7-DOUT) -> Net-(D7-A)
- D8 pad 1: +5V -> unconnected-(D8A-A1-Pad1)
- D8 pad 2: Net-(D8-DOUT) -> +3V3_ANA
- D8 pad 3: GND -> (no net)
- D8 pad 4: Net-(D7-DOUT) -> (no net)
- D9 pad 2: Net-(D10-DIN) -> Net-(D11-DIN)
- D9 pad 4: Net-(D8-DOUT) -> Net-(D9-DIN)
- FB1 pad 1: +5V -> Net-(D4-A1)
- FB1 pad 2: Net-(D2-A1) -> +5V
- J1 pad 1: Net-(D1-A) -> GND
- J1 pad 2: GND -> /Power & USB/preVBUS
- J2 pad 1: Net-(D1-A) -> /Power & USB/preVBUS
- J3 pad 2: Net-(J3-D-) -> DM
- J3 pad 3: Net-(J3-D+) -> DP
- J4 pad 1: /VGA/VGA_R -> Net-(165_4-D0)
- J4 pad 2: /VGA/VGA_G -> Net-(165_4-D1)
- J5 pad 1: Net-(165_1-D0) -> /ADC/ANALOG_IN
- J5 pad 2: Net-(165_1-D1) -> Net-(J5-Pin_2)
- J6 pad 1: /ADC/ANALOG_IN -> /VGA/VGA_R
- J6 pad 2: Net-(J6-Pin_2) -> /VGA/VGA_G
- J6 pad 3: Net-(J6-Pin_3) -> /VGA/VGA_B
- J7 pad 1: unconnected-(J7-Pin_1-Pad1) -> GND
- J7 pad 2: unconnected-(J7-Pin_2-Pad2) -> +3V3
- J7 pad 3: unconnected-(J7-Pin_3-Pad3) -> SDA
- J7 pad 4: unconnected-(J7-Pin_4-Pad4) -> SCL
- J7 pad 5: GND -> (no net)
- J7 pad 6: +3V3 -> (no net)
- JP1 pad 1: Net-(D3-K) -> GND
- JP1 pad 2: +5V_UP -> Net-(JP1-C)
- LED1 pad 1: GND -> unconnected-(LED1-K-Pad1)
- LED1 pad 2: Net-(LED1-A) -> unconnected-(LED1-A-Pad2)
- LED3 pad 1: unconnected-(LED3-K-Pad1) -> GND
- LED3 pad 2: unconnected-(LED3-A-Pad2) -> Net-(LED3-A)
- Q2 pad 3: /Output Chain/SEG_CA1 -> /Output Chain/SEG_CA2
- Q4 pad 3: /Output Chain/SEG_CA2 -> /Output Chain/SEG_CA4
- R1 pad 1: GND -> SDA
- R1 pad 2: /Input Chain/BTN_LEFT -> +3V3
- R10 pad 1: VGA_R0 -> Net-(U2-IOB_29B)
- R10 pad 2: /VGA/VGA_R -> SPI_CS_ADC
- R109 pad 1: unconnected-(R109-Pad1) -> Net-(R107-Pad2)
- R109 pad 2: SPI_MISO -> Net-(R108-Pad2)
- R11 pad 1: VGA_R1 -> Net-(U2-IOB_22A)
- R11 pad 2: /VGA/VGA_R -> PMOD_7
- R110 pad 1: unconnected-(R110-Pad1) -> Net-(R107-Pad2)
- R110 pad 2: SPI_MOSI -> Net-(R110-Pad2)
- R111 pad 1: unconnected-(R111-Pad1) -> Net-(R110-Pad2)
- R111 pad 2: SPI_SCK -> GND
- R112 pad 1: unconnected-(R112-Pad1) -> +3V3
- R112 pad 2: SPI_CS_ADC -> SPI_CS_DAC
- R113 pad 1: unconnected-(R113-Pad1) -> VGA_R0
- R113 pad 2: SPI_CS_DAC -> /VGA/VGA_R
- R114 pad 1: unconnected-(R114-Pad1) -> VGA_R1
- R114 pad 2: SIN_DOUT -> /VGA/VGA_R
- R115 pad 1: unconnected-(R115-Pad1) -> VGA_R2
- R115 pad 2: SIN_SCLK -> /VGA/VGA_R
- R116 pad 1: unconnected-(R116-Pad1) -> VGA_G0
- R116 pad 2: SOUT_DIN -> /VGA/VGA_G
- R117 pad 1: unconnected-(R117-Pad1) -> VGA_G1
- R117 pad 2: SIN_SHLD -> /VGA/VGA_G
- R118 pad 1: unconnected-(R118-Pad1) -> VGA_G2
- R118 pad 2: SOUT_RCLK -> /VGA/VGA_G
- R119 pad 1: unconnected-(R119-Pad1) -> VGA_B0
- R119 pad 2: TX -> /VGA/VGA_B
- R12 pad 1: VGA_R2 -> Net-(U2-IOB_24A)
- R12 pad 2: /VGA/VGA_R -> PMOD_9
- R120 pad 1: unconnected-(R120-Pad1) -> VGA_B1
- R120 pad 2: SOUT_SCLK -> /VGA/VGA_B
- R121 pad 1: unconnected-(R121-Pad1) -> VGA_B2
- R121 pad 2: WS_DIN -> /VGA/VGA_B
- R122 pad 1: /BTN0 -> Net-(C24-Pad2)
- R122 pad 2: Net-(BTN0-Pad2) -> GND
- R123 pad 1: unconnected-(R123-Pad1) -> /VGA/_VGA_HS
- R123 pad 2: RX -> VGA_HS
- R124 pad 1: unconnected-(R124-Pad1) -> /VGA/_VGA_VS
- R124 pad 2: /SCL -> VGA_VS
- R125 pad 1: unconnected-(R125-Pad1) -> Net-(R125-Pad1)
- R125 pad 2: /SDA -> Net-(D9-DIN)
- R13 pad 1: VGA_G0 -> Net-(U2-IOB_31B)
- R13 pad 2: /VGA/VGA_G -> SPI_CS_DAC
- R14 pad 1: VGA_G1 -> Net-(U2-IOB_0A)
- R14 pad 2: /VGA/VGA_G -> SOUT_SCLK
- R15 pad 1: VGA_G2 -> Net-(U2-IOB_2A)
- R15 pad 2: /VGA/VGA_G -> SOUT_DIN
- R16 pad 1: VGA_B0 -> Net-(U2-IOB_6A)
- R16 pad 2: /VGA/VGA_B -> SOUT_RCLK
- R17 pad 1: VGA_B1 -> Net-(U2-IOB_9B)
- R17 pad 2: /VGA/VGA_B -> UART_RX
- R18 pad 1: VGA_B2 -> Net-(U2-IOB_4A)
- R18 pad 2: /VGA/VGA_B -> UART_TX
- R19 pad 2: +3V3 -> /CLK_12M_EXT
- R2 pad 1: GND -> SCL
- R2 pad 2: /Input Chain/BTN_UP -> +3V3
- R20 pad 1: GND -> Net-(R20-Pad1)
- R20 pad 2: Net-(BTN0-Pad2) -> /IOB_25B_G3
- R21 pad 1: /Input Chain/ENC_SW -> Net-(J3-Shield)
- R21 pad 2: +3V3 -> GND
- R22 pad 1: Net-(C5-Pad2) -> UART_TX
- R22 pad 2: GND -> +3V3
- R23 pad 1: /VGA/_VGA_HS -> UART_RX
- R23 pad 2: VGA_HS -> +3V3_UP
- R24 pad 1: /VGA/_VGA_VS -> Net-(D6-A)
- R24 pad 2: VGA_VS -> +5V
- R25 pad 1: TX -> Net-(D7-A)
- R26 pad 1: RX -> /Input Chain/KB_ROW1
- R26 pad 2: +3V3_UP -> GND
- R27 pad 1: /SDA -> GND
- R27 pad 2: +3V3 -> /Input Chain/KB_ROW2
- R28 pad 1: /SCL -> /Input Chain/KB_ROW3
- R28 pad 2: +3V3 -> GND
- R29 pad 1: Net-(R29-Pad1) -> GND
- R29 pad 2: Net-(D5-DIN) -> /Input Chain/KB_ROW4
- R3 pad 1: GND -> Net-(U2-IOT_51A)
- R3 pad 2: /Input Chain/BTN_CENTER -> SIN_DOUT
- R31 pad 2: /Input Chain/SEL_1 -> /Input Chain/BTN_LEFT
- R32 pad 1: Net-(165_1-D0) -> GND
- R32 pad 2: +3V3 -> /Input Chain/SEL_1
- R33 pad 1: Net-(165_1-D1) -> Net-(R33-Pad1)
- R33 pad 2: +3V3 -> /Input Chain/ENC_A
- R34 pad 1: /Input Chain/KB_ROW1 -> Net-(R34-Pad1)
- R34 pad 2: GND -> /Input Chain/ENC_B
- R35 pad 1: GND -> Net-(R33-Pad1)
- R35 pad 2: /Input Chain/KB_ROW2 -> +3V3
- R36 pad 1: /Input Chain/KB_ROW3 -> Net-(R34-Pad1)
- R36 pad 2: GND -> +3V3
- R37 pad 2: /Input Chain/KB_ROW4 -> /Input Chain/BTN_UP
- R38 pad 1: /Output Chain/SEG_A -> GND
- R38 pad 2: Net-(595_2-QH) -> /Input Chain/BTN_CENTER
- R39 pad 1: /Output Chain/SEG_B -> GND
- R39 pad 2: Net-(595_2-QG) -> /Input Chain/BTN_DOWN
- R4 pad 1: GND -> Net-(U2-IOT_41A)
- R4 pad 2: /Input Chain/BTN_DOWN -> SIN_SCLK
- R40 pad 1: /Output Chain/SEG_C -> /Input Chain/ENC_SW
- R40 pad 2: Net-(595_2-QF) -> +3V3
- R41 pad 1: /Output Chain/SEG_D -> GND
- R41 pad 2: Net-(595_2-QE) -> /Input Chain/BTN_RIGHT
- R42 pad 1: /Output Chain/SEG_E -> Net-(165_4-D1)
- R42 pad 2: Net-(595_2-QD) -> +3V3
- R43 pad 1: /Output Chain/SEG_F -> Net-(165_4-D0)
- R43 pad 2: Net-(595_2-QC) -> +3V3
- R44 pad 1: /Output Chain/SEG_G -> /Output Chain/KB_COL1
- R44 pad 2: Net-(595_2-QB) -> Net-(595_1-QA)
- R45 pad 1: /Output Chain/SEG_DP -> /Output Chain/KB_COL2
- R45 pad 2: Net-(595_2-QA) -> Net-(595_1-QB)
- R46 pad 1: Net-(LED0-A) -> /Output Chain/KB_COL3
- R46 pad 2: Net-(595_3-QA) -> Net-(595_1-QC)
- R47 pad 1: Net-(LED1-A) -> /Output Chain/KB_COL4
- R47 pad 2: Net-(595_3-QB) -> Net-(595_1-QD)
- R48 pad 1: Net-(LED2-A) -> /Output Chain/SEG_DP
- R48 pad 2: Net-(595_3-QC) -> Net-(595_2-QA)
- R49 pad 1: unconnected-(R49-Pad1) -> /Output Chain/SEG_G
- R49 pad 2: Net-(595_3-QD) -> Net-(595_2-QB)
- R5 pad 1: GND -> Net-(U2-IOT_50B)
- R5 pad 2: /Input Chain/BTN_RIGHT -> SIN_SHLD
- R50 pad 1: Net-(LED4-A) -> /Output Chain/SEG_F
- R50 pad 2: Net-(595_3-QE) -> Net-(595_2-QC)
- R51 pad 1: Net-(LED5-A) -> /Output Chain/SEG_E
- R51 pad 2: Net-(595_3-QF) -> Net-(595_2-QD)
- R52 pad 1: Net-(LED6-A) -> /Output Chain/SEG_D
- R52 pad 2: Net-(595_3-QG) -> Net-(595_2-QE)
- R53 pad 1: Net-(LED7-A) -> /Output Chain/SEG_C
- R53 pad 2: Net-(595_3-QH) -> Net-(595_2-QF)
- R54 pad 1: Net-(LED8-A) -> /Output Chain/SEG_B
- R54 pad 2: Net-(595_4-QA) -> Net-(595_2-QG)
- R55 pad 1: Net-(LED9-A) -> /Output Chain/SEG_A
- R55 pad 2: Net-(595_4-QB) -> Net-(595_2-QH)
- R56 pad 1: Net-(LED10-A) -> Net-(Q1-B)
- R56 pad 2: Net-(595_4-QC) -> /Output Chain/preSEG_CA1
- R57 pad 1: Net-(LED11-A) -> Net-(Q2-B)
- R57 pad 2: Net-(595_4-QD) -> /Output Chain/preSEG_CA2
- R58 pad 1: Net-(LED12-A) -> Net-(Q3-B)
- R58 pad 2: Net-(595_4-QE) -> /Output Chain/preSEG_CA3
- R59 pad 1: Net-(LED13-A) -> Net-(Q4-B)
- R59 pad 2: Net-(595_4-QF) -> /Output Chain/preSEG_CA4
- R6 pad 1: Net-(R6-Pad1) -> GND
- R6 pad 2: /Input Chain/ENC_A -> Net-(BTN1-Pad2)
- R60 pad 1: Net-(LED14-A) -> Net-(LED2-A)
- R60 pad 2: Net-(595_4-QG) -> Net-(595_3-QA)
- R61 pad 1: Net-(LED15-A) -> Net-(LED3-A)
- R61 pad 2: Net-(595_4-QH) -> Net-(595_3-QB)
- R62 pad 1: Net-(Q2-B) -> Net-(LED4-A)
- R62 pad 2: /Output Chain/preSEG_CA1 -> Net-(595_3-QC)
- R63 pad 1: Net-(Q3-B) -> unconnected-(R63-Pad1)
- R63 pad 2: /Output Chain/preSEG_CA3 -> Net-(595_3-QD)
- R64 pad 1: Net-(Q4-B) -> Net-(LED5-A)
- R64 pad 2: /Output Chain/preSEG_CA2 -> Net-(595_3-QE)
- R65 pad 1: Net-(Q5-B) -> Net-(LED6-A)
- R65 pad 2: /Output Chain/preSEG_CA4 -> Net-(595_3-QF)
- R66 pad 1: /Output Chain/KB_COL1 -> Net-(LED7-A)
- R66 pad 2: Net-(595_1-QA) -> Net-(595_3-QG)
- R67 pad 1: /Output Chain/KB_COL2 -> Net-(LED8-A)
- R67 pad 2: Net-(595_1-QB) -> Net-(595_3-QH)
- R68 pad 1: /Output Chain/KB_COL3 -> Net-(LED9-A)
- R68 pad 2: Net-(595_1-QC) -> Net-(595_4-QA)
- R69 pad 1: /Output Chain/KB_COL4 -> Net-(LED10-A)
- R69 pad 2: Net-(595_1-QD) -> Net-(595_4-QB)
- R7 pad 1: Net-(R19-Pad1) -> /BTN0
- R7 pad 2: /Input Chain/ENC_B -> Net-(BTN1-Pad2)
- R70 pad 1: Net-(U8-+) -> Net-(LED11-A)
- R70 pad 2: Net-(595_5-QA) -> Net-(595_4-QC)
- R71 pad 1: Net-(R71-Pad1) -> Net-(LED12-A)
- R71 pad 2: Net-(595_5-QB) -> Net-(595_4-QD)
- R72 pad 1: Net-(U8-+) -> Net-(LED13-A)
- R72 pad 2: Net-(R71-Pad1) -> Net-(595_4-QE)
- R73 pad 1: Net-(R73-Pad1) -> Net-(LED14-A)
- R73 pad 2: Net-(595_5-QC) -> Net-(595_4-QF)
- R74 pad 1: Net-(R74-Pad1) -> Net-(LED15-A)
- R74 pad 2: Net-(595_5-QD) -> Net-(595_4-QG)
- R75 pad 1: Net-(R75-Pad1) -> Net-(LED16-A)
- R75 pad 2: Net-(595_5-QE) -> Net-(595_4-QH)
- R76 pad 1: Net-(R76-Pad1) -> Net-(U6-Tip)
- R76 pad 2: Net-(595_5-QF) -> /ADC/AUDIO_IN
- R77 pad 1: Net-(R77-Pad1) -> Net-(U6-Ring1)
- R77 pad 2: Net-(595_5-QG) -> /ADC/AUDIO_IN
- R78 pad 1: Net-(R78-Pad1) -> +3V3_ANA
- R78 pad 2: Net-(595_5-QH) -> Net-(J5-Pin_3)
- R79 pad 1: Net-(R71-Pad1) -> Net-(J5-Pin_3)
- R79 pad 2: Net-(R73-Pad1) -> GND
- R8 pad 1: Net-(J3-Shield) -> Net-(U2-IOB_5B)
- R8 pad 2: GND -> WS_DIN
- R80 pad 1: Net-(R73-Pad1) -> +3V3_ANA
- R80 pad 2: Net-(R74-Pad1) -> /ADC/ADC_CH2
- R81 pad 1: Net-(R74-Pad1) -> /ADC/ADC_CH2
- R81 pad 2: Net-(R75-Pad1) -> GND
- R82 pad 1: Net-(R75-Pad1) -> /ADC/ADC_CH0
- R82 pad 2: Net-(R76-Pad1) -> Net-(R82-Pad2)
- R83 pad 1: Net-(R76-Pad1) -> Net-(J5-Pin_2)
- R83 pad 2: Net-(R77-Pad1) -> Net-(D8A-K3A4)
- R84 pad 1: Net-(R77-Pad1) -> Net-(D8A-K3A4)
- R84 pad 2: Net-(R78-Pad1) -> /ADC/ADC_CH1
- R85 pad 1: Net-(R78-Pad1) -> PMOD_9
- R85 pad 2: GND -> +3V3
- R87 pad 1: Net-(J6-Pin_2) -> Net-(595_5-QA)
- R87 pad 2: Net-(D22-A) -> Net-(R87-Pad2)
- R88 pad 1: Net-(J6-Pin_3) -> Net-(U8-+)
- R88 pad 2: GND -> Net-(R87-Pad2)
- R89 pad 1: +3V3_ANA -> Net-(U8-+)
- R89 pad 2: Net-(J6-Pin_3) -> Net-(R89-Pad2)
- R9 pad 1: Net-(R6-Pad1) -> Net-(U2-IOB_23B)
- R9 pad 2: +3V3 -> PMOD_8
- R90 pad 1: +3V3_ANA -> Net-(595_5-QB)
- R90 pad 2: /ADC/ADC_CH2 -> Net-(R90-Pad2)
- R91 pad 1: /ADC/ADC_CH2 -> Net-(R89-Pad2)
- R91 pad 2: GND -> Net-(R90-Pad2)
- R92 pad 1: SPI_SCK -> Net-(R89-Pad2)
- R92 pad 2: +3V3 -> Net-(R92-Pad2)
- R93 pad 1: +3V3 -> Net-(595_5-QC)
- R93 pad 2: SPI_CS_DAC -> Net-(R93-Pad2)
- R94 pad 1: Net-(D24-A) -> Net-(R92-Pad2)
- R94 pad 2: +5V -> Net-(R93-Pad2)
- R95 pad 1: Net-(D25-A) -> Net-(R92-Pad2)
- R95 pad 2: +3V3 -> Net-(R95-Pad2)
- R96 pad 1: /ADC/ADC_CH0 -> Net-(595_5-QD)
- R97 pad 1: Net-(D22-A) -> Net-(R95-Pad2)
- R97 pad 2: /ADC/ADC_CH1 -> Net-(R96-Pad2)
- R98 pad 1: Net-(U9-Tip) -> Net-(R95-Pad2)
- R98 pad 2: /ADC/AUDIO_IN -> Net-(R100-Pad1)
- R99 pad 1: Net-(U9-Ring1) -> Net-(595_5-QE)
- R99 pad 2: /ADC/AUDIO_IN -> Net-(R100-Pad2)
- RV1 pad 2: Net-(R96-Pad2) -> Net-(R82-Pad2)
- TH1 pad 1: Net-(D2-A1) -> Net-(D4-A1)
- TP14 pad 1: GND -> +5V
- TP15 pad 1: GND -> UART_RX
- TP2 pad 1: Net-(D1-A) -> +3V3_UP
- TP23 pad 1: GND -> /ADC/AUDIO_IN
- TP24 pad 1: GND -> /ADC/ANALOG_IN
- TP25 pad 1: RX -> /ADC/AUDIO_IN
- TP26 pad 1: TX -> /ADC/ADC_CH0
- TP27 pad 1: Net-(J3-D-) -> DAC_OUT
- TP28 pad 1: Net-(J3-D+) -> /ADC/ADC_CH2
- TP29 pad 1: VBUS -> /ADC/ADC_CH1
- TP3 pad 1: GND -> SDA
- TP30 pad 1: +5V -> DAC_OUT
- TP31 pad 1: +3V3 -> RDAC_OUT
- TP32 pad 1: +3V3_ANA -> DAC_OUT
- TP33 pad 1: /VGA/_VGA_VS -> RDAC_OUT
- TP34 pad 1: /VGA/_VGA_HS -> Net-(U8-+)
- TP35 pad 1: /VGA/VGA_B -> /VGA/VGA_R
- TP37 pad 1: /VGA/VGA_R -> /VGA/VGA_B
- TP38 pad 1: +5V_UP -> /VGA/_VGA_HS
- TP39 pad 1: +3V3_UP -> /VGA/_VGA_VS
- TP4 pad 1: /ADC/AUDIO_IN -> SCL
- TP40 pad 1: /ADC/AUDIO_IN -> WS_DIN
- TP41 pad 1: /ADC/ANALOG_IN -> Net-(R125-Pad1)
- TP42 pad 1: /ADC/ADC_CH0 -> Net-(D10-DOUT)
- TP43 pad 1: /ADC/ADC_CH1 -> Net-(D17-DOUT)
- TP6 pad 1: /ADC/ANALOG_IN -> Net-(R19-Pad1)
- TP7 pad 1: RDAC_OUT -> Net-(R20-Pad1)
- TP8 pad 1: DAC_OUT -> GND
- U1 pad 1: /Output Chain/SEG_E -> GND
- U1 pad 2: /Output Chain/SEG_D -> GND
- U1 pad 3: /Output Chain/SEG_DP -> GND
- U1 pad 4: /Output Chain/SEG_C -> GND
- U1 pad 5: /Output Chain/SEG_G -> SDA
- U1 pad 6: /Output Chain/SEG_CA4 -> SCL
- U1 pad 7: /Output Chain/SEG_B -> Net-(JP1-C)
- U1 pad 8: /Output Chain/SEG_CA3 -> +3V3
- U2 pad 1: Net-(J3-D+) -> GND
- U2 pad 2: Net-(J3-D-) -> unconnected-(U2-VIO_BANK_0_2-Pad2)
- U2 pad 3: GND -> unconnected-(U2-CRESET_N-Pad3)
- U2 pad 5: +3V3 -> unconnected-(U2-LED_R-Pad5)
- U2 pad 6: Net-(D4-K) -> unconnected-(U2-LED_G-Pad6)
- U2 pad 7: TX -> unconnected-(U2-LED_B-Pad7)
- U2 pad 8: +3V3 -> +5V_UP
- U3 pad 1: GND -> +5V
- U3 pad 3: GND -> +5V
- U3 pad 4: GND -> unconnected-(U3-NC-Pad4)
- U3 pad 5: /SDA -> +3V3
- U4 pad 1: /ADC/ADC_CH0 -> DP
- U4 pad 2: /ADC/ADC_CH1 -> DM
- U4 pad 3: /ADC/ADC_CH2 -> GND
- U4 pad 4: DAC_OUT -> unconnected-(U4-~{RTS}-Pad4)
- U4 pad 5: unconnected-(U4-NC-Pad5) -> +3V3
- U4 pad 6: unconnected-(U4-NC-Pad6) -> Net-(D5-K)
- U4 pad 7: GND -> UART_TX
- U4 pad 8: SPI_SCK -> +3V3
- U5 pad 1: +5V -> /Output Chain/SEG_E
- U5 pad 2: GND -> /Output Chain/SEG_D
- U5 pad 3: +5V -> /Output Chain/SEG_DP
- U5 pad 4: unconnected-(U5-NC-Pad4) -> /Output Chain/SEG_C
- U5 pad 5: +3V3 -> /Output Chain/SEG_G
- U6 pad 2: WS_DIN -> Net-(U6-Tip)
- U6 pad 3: GND -> Net-(U6-Ring1)
- U6 pad 4: Net-(R29-Pad1) -> unconnected-(U6-Ring2-Pad4)
- U7 pad 1: GND -> /ADC/ADC_CH0
- U7 pad 10: GND -> PMOD_7
- U7 pad 11: unconnected-(U7-IOT_37A-Pad11) -> SPI_CS_ADC
- U7 pad 12: unconnected-(U7-IOT_36B-Pad12) -> GND
- U7 pad 13: unconnected-(U7-IOT_39A-Pad13) -> +3V3_ANA
- U7 pad 14: unconnected-(U7-IOT_38B-Pad14) -> +3V3_ANA
- U7 pad 2: unconnected-(U7-VIO_BANK_0_2-Pad2) -> /ADC/ADC_CH1
- U7 pad 3: /nRST_UP -> /ADC/ADC_CH2
- U7 pad 4: unconnected-(U7-CDONE-Pad4) -> DAC_OUT
- U7 pad 7: unconnected-(U7-LED_B-Pad7) -> GND
- U7 pad 8: +5V_UP -> PMOD_9
- U7 pad 9: +3V3_UP -> PMOD_8
- U9 pad 2: Net-(U9-Tip) -> WS_DIN
- U9 pad 3: Net-(U9-Ring1) -> GND
- U9 pad 4: unconnected-(U9-Ring2-Pad4) -> Net-(R125-Pad1)
Routing:
- net /Power & USB/preVBUS: track 0.00 -> 25.2 mm
- net GND: track 0.00 -> 11.9 mm, vias 0 -> 2
- net /VGA/VGA_G: track 0.00 -> 6.59 mm, vias 0 -> 1
- net PMOD_3: track 0.00 -> 4.91 mm
- added copper zone on In1.Cu, net GND
Other:
- board outline added: 150 x 150 mm
- copper layers 2 -> 4
