File: hardware/gatebench.kicad_sch (KiCad schematic)
At the start: 33 parts, among them J7 PMOD, J9 Qwiic | STEMMA QT, U3 24LC02, U7 UPduinoV3_1Board

Commit message: feat(hw): closing sch, starting pcb
Parts:
- removed J7: PMOD, Connector_PinHeader_2.54mm:PinHeader_2x06_P2.54mm_Horizontal, symbol Connector_Generic:Conn_02x06_Top_Bottom
- removed J9: Qwiic | STEMMA QT, CONN_SM04B_JST, symbol SM04B-SRSS-TB:SM04B-SRSS-TBLFSN
- removed R109, R110, R111, R112, R113, R114, R115, R116, R117, R118, R120, R121, R124, R125: 100, Resistor_SMD:R_0603_1608Metric, symbol Device:R
- added D1: BAV199DW, Package_TO_SOT_SMD:SOT-363_SC-70-6, symbol Diode:BAV199DW
- added H1, H2, H3, H4: MountingHole, MountingHole:MountingHole_3.2mm_M3, symbol Mechanical:MountingHole
- added JP2: Jumper_2_Open, symbol Jumper:Jumper_2_Open
- added R10, R11, R12, R13, R14, R15, R16, R19, R20, R3, R4, R5, R8, R9: 100, Resistor_SMD:R_0603_1608Metric, symbol Device:R
- added TP5, TP6, TP7: TestPoint_Alt, Connector_PinHeader_2.54mm:PinHeader_1x01_P2.54mm_Vertical, symbol Connector:TestPoint_Alt
- renumbered BTN0 to BTN1, C7 to C1, C13 to C2, C14 to C3, JP2 to JP1, R27 to R1, R123 to R17, R119 to R18, R28 to R2, R20 to R6, R122 to R7, TP38 to TP1, TP39 to TP2, TP53 to TP3, TP54 to TP4, U3 to U1, U7 to U2
Connections:
- net +3V3: now also D1.2 (K2)
- net BTN0: now also U2.31 (IOB_8A)
- net GND: now also D1.1 (A1)
- net SCL: now also U2.32 (IOB_3B_G6)
- net SDA: now also U2.33 (IOB_13B)
- net SIN_DOUT: now also R3.2
- net SIN_SCLK: now also R4.2
- net SIN_SHLD: now also R5.2
- net SOUT_DIN: now also R15.2
- net SOUT_RCLK: now also R16.2
- net SOUT_SCLK: now also R14.2
- net SPI_CS_ADC: now also R10.2
- net SPI_CS_DAC: now also R13.2
- net SPI_MISO: now also R11.2
- net SPI_MOSI: now also R9.2
- net SPI_SCK: now also R12.2
- net VGA_B0: now also U2.17 (IOT_42B)
- net VGA_B1: now also U2.18 (IOT_45A_G1)
- net VGA_B2: now also U2.19 (IOT_44B)
- net VGA_G0: now also U2.14 (IOT_38B)
- net VGA_G1: now also U2.15 (IOT_43A)
- net VGA_G2: now also U2.16 (IOT_46B_G0)
- net VGA_HS: now also U2.20 (IOT_49A)
- net VGA_R0: now also U2.11 (IOT_37A)
- net VGA_R1: now also U2.12 (IOT_36B)
- net VGA_R2: now also U2.13 (IOT_39A)
- net VGA_VS: now also U2.21 (IOT_48B)
- net WS_DIN: now also R8.2
- net at BTN1.2, R6.2, R7.2: now also TP5.1
- net at R17.1: now also U2.30 (IOB_9B)
- net at R18.1: now also U2.29 (IOB_4A)
- net at U2.22 (IOT_51A): now also R3.1
- net at U2.23 (IOT_50B): now also R5.1
- net at U2.24 (IOT_41A): now also R4.1
- net at U2.25 (IOB_6A): now also R16.1
- net at U2.26 (IOB_0A): now also R14.1
- net at U2.27 (IOB_2A): now also R15.1
- net at U2.28 (IOB_5B): now also R8.1
- net PMOD_4: now reaches U2.34 (IOB_16A)
- net PMOD_3: now reaches U2.35 (IOB_20A)
- net at U2.36 (IOB_31B): now also R13.1
- net at U2.37 (IOB_29B): now also R10.1
- net at U2.38 (IOB_24A): now also R12.1
- net at U2.39 (IOB_23B): now also R9.1
- net at U2.40 (IOB_22A): now also R11.1
- net CLK_12M_EXT: now reaches U2.41 (CLK_12M_EXT)
- net CLK_12M_EXT: now also D1.6 (K3A4), JP2.1 (A), R19.2
- net PMOD_2: now reaches U2.43 (IOB_18A)
- net IOB_25B_G3: now reaches U2.44 (IOB_25B_G3)
- net IOB_25B_G3: now also JP2.2 (B), R20.2
- net nRST_UP: no longer names the net of U2.3 (CRESET_N)
- new net: R19.1, TP6.1
- new net: R20.1, TP7.1
- no-connect marks 0 -> 10
Other:
- added sheet Expansion (expansion.kicad_sch)
- moved on the sheet: BTN1, C1, C2, C3, JP1, R1, R17, R18, R2, R6, R7, TP1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
