File: hardware/inputchain.kicad_sch (KiCad schematic)
At the start: 49 parts, among them J5 Conn_01x02_Pin, SW1 SW_SPDT, SW10 SW_SPDT, SW11 SW_SPDT, SW12 SW_SPDT, SW13 SW_SPDT, SW14 SW_SPDT, SW15 SW_SPDT, SW16 SW_SPDT, SW17 RotaryEncoder, SW18 SW_DIP_x02, SW2 SW_SPDT, SW3 SW_SPDT, SW4 SW_SPDT, SW5 SW_SPDT, SW6 SW_SPDT, SW7 SW_SPDT, SW8 SW_SPDT, SW9 SW_SPDT

Commit message: feat(hw): closing sch, starting pcb
Parts:
- renumbered 165_3 to 165_1, 165_4 to 165_2, 165_2 to 165_3, 165_1 to 165_4, C1 to C12, C2 to C13, J5 to J4, R34 to R26, R35 to R27, R36 to R28, R37 to R29, R1 to R31, R31 to R32, R6 to R33, R7 to R34, R9 to R35, R19 to R36, R2 to R37, R3 to R38, R4 to R39, R21 to R40, R5 to R41, R33 to R42, R32 to R43, SW18 to SW17, SW17 to SW18
