File: hardware/outputchain.kicad_sch (KiCad schematic)
At the start: 57 parts, among them Q2 MMBT3906, Q3 MMBT3906, Q4 MMBT3906, Q5 MMBT3906, U1 CA56-12EWA

Commit message: feat(hw): closing sch, starting pcb
Parts:
- renumbered LED3 to LED1, LED9 to LED10, LED10 to LED11, LED11 to LED12, LED12 to LED13, LED13 to LED14, LED14 to LED15, LED15 to LED16, LED0 to LED2, LED1 to LED3, LED2 to LED4, LED4 to LED5, LED5 to LED6, LED6 to LED7, LED7 to LED8, LED8 to LED9, Q2 to Q1, Q4 to Q2, Q5 to Q4, R66 to R44, R67 to R45, R68 to R46, R69 to R47, R45 to R48, R44 to R49, R43 to R50, R42 to R51, R41 to R52, R40 to R53, R39 to R54, R38 to R55, R62 to R56, R64 to R57, R63 to R58, R65 to R59, R46 to R60, R47 to R61, R48 to R62, R49 to R63, R50 to R64, R51 to R65, R52 to R66, R53 to R67, R54 to R68, R55 to R69, R56 to R70, R57 to R71, R58 to R72, R59 to R73, R60 to R74, R61 to R75, U1 to U5
