File: hardware/powernusb.kicad_sch (KiCad schematic)
At the start: 42 parts, among them J1 Conn_01x02_Pin, J2 Screw_Terminal_01x02, J3 USB_B, U2 CH340N, U5 AP2112K-3.3

Commit message: feat(hw): closing sch, starting pcb
Parts:
- removed D2: SMF5V0A, Diode_SMD:D_SMF, symbol Diode:SMF5V0A
- removed TP30: TestPoint_Alt, Connector_PinHeader_2.54mm:PinHeader_1x01_P2.54mm_Vertical, symbol Connector:TestPoint_Alt
- added D4: SMF5V0A, Diode_SMD:D_SMF, symbol Diode:SMF5V0A
- added TP14: TestPoint_Alt, Connector_PinHeader_2.54mm:PinHeader_1x01_P2.54mm_Vertical, symbol Connector:TestPoint_Alt
- D3: renamed from D1; footprint Package_TO_SOT_SMD:SOT-583-8 -> Diode_SMD:Nexperia_CFP3_SOD-123W
- R22: renamed from R25; now not fitted
- renumbered C19 to C10, C20 to C11, C3 to C4, C8 to C5, C9 to C6, C10 to C7, C6 to C8, C11 to C9, D3 to D2, D4 to D5, D24 to D6, D25 to D7, JP1 to JP3, R8 to R21, R26 to R23, R94 to R24, R95 to R25, TP29 to TP10, TP27 to TP11, TP28 to TP12, TP31 to TP13, TP25 to TP15, TP26 to TP16, TP32 to TP17, TP14 to TP18, TP24 to TP19, TP15 to TP20, TP23 to TP21, TP3 to TP8, TP2 to TP9, U5 to U3, U2 to U4
Connections:
- net +5V: now also FB1.2, TP14.1; no longer FB1.1
- net GND: now also J1.1 (Pin_1), D4.2 (A2); no longer J1.2 (Pin_2)
- net preVBUS: now reaches D3.2 (A), J2.1 (Pin_1), TP9.1
- net preVBUS: now also J1.2 (Pin_2); no longer J1.1 (Pin_1)
- net at TH1.1: now also FB1.1, D4.1 (A1); no longer FB1.2
- net DM: now reaches J3.2 (D-), TP11.1, U4.2 (UD-)
- net DP: now reaches J3.3 (D+), TP12.1, U4.1 (UD+)
- no-connect marks 0 -> 1
Other:
- note added: "Connected to driver's RXD"
- note added: "Connected to driver's TXD"
- moved on the sheet: TH1, TP11, TP12
