File: hardware/vga.kicad_sch (KiCad schematic)
At the start: 19 parts, among them J4 DE15_Socket_HighDensity_Mount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

Commit message: feat(hw): closing sch, starting pcb
Parts:
- renumbered C5 to C24, J4 to J6, R10 to R113, R11 to R114, R12 to R115, R13 to R116, R14 to R117, R15 to R118, R16 to R119, R17 to R120, R18 to R121, R22 to R122, R23 to R123, R24 to R124, TP37 to TP35, TP35 to TP37, TP34 to TP38, TP33 to TP39
Changed lines of the file:
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@@
 		(dnp no)
 		(fields_autoplaced yes)
-		(property "Reference" "#PWR068"
+		(property "Reference" "#PWR0177"
 			(at 175.26 121.92 0)
 			(hide yes)
@@
 			(project "gatebench"
 				(path "/f24451ff-caac-4926-9774-6edc1451b63f/a3c4557c-c544-4f42-ade0-8584472233ea"
-					(reference "#PWR068")
+					(reference "#PWR0177")
 					(unit 1)
 				)
@@
 		(in_pos_files yes)
 		(dnp no)
-		(property "Reference" "R15"
+		(property "Reference" "R118"
 			(at 124.46 93.218 90)
 			(show_name no)
@@
 			(project "gatebench"
 				(path "/f24451ff-caac-4926-9774-6edc1451b63f/a3c4557c-c544-4f42-ade0-8584472233ea"
-					(reference "R15")
+					(reference "R118")
 					(unit 1)
 				)
@@
 		(in_pos_files yes)
 		(dnp no)
-		(property "Reference" "R12"
+		(property "Reference" "R115"
 			(at 124.46 75.438 90)
 			(show_name no)
@@
 			(project "gatebench"
 				(path "/f24451ff-caac-4926-9774-6edc1451b63f/a3c4557c-c544-4f42-ade0-8584472233ea"
-					(reference "R12")
+					(reference "R115")
 					(unit 1)
 				)
@@
 		(in_pos_files yes)
 		(dnp no)
-		(property "Reference" "J4"
+		(property "Reference" "J6"
 			(at 157.48 75.692 0)
 			(show_name no)
@@
 			(project "gatebench"
 				(path "/f24451ff-caac-4926-9774-6edc1451b63f/a3c4557c-c544-4f42-ade0-8584472233ea"
-					(reference "J4")
+					(reference "J6")
 					(unit 1)
 				)
@@
 		(in_pos_files yes)
 		(dnp no)
-		(property "Reference" "C5"
+		(property "Reference" "C24"
 			(at 166.37 123.19 90)
 			(show_name no)
@@
 			(project "gatebench"
 				(path "/f24451ff-caac-4926-9774-6edc1451b63f/a3c4557c-c544-4f42-ade0-8584472233ea"
-					(reference "C5")
+					(reference "C24")
 					(unit 1)
 				)
@@
 		(in_pos_files yes)
 		(dnp no)
-		(property "Reference" "TP35"
+		(property "Reference" "TP37"
 			(at 214.122 54.61 90)
 			(show_name no)
@@
 			(project "gatebench"
 				(path "/f24451ff-caac-4926-9774-6edc1451b63f/a3c4557c-c544-4f42-ade0-8584472233ea"
-					(reference "TP35")
+					(reference "TP37")
 					(unit 1)
 				)
@@
 		(in_pos_files yes)
 		(dnp no)
-		(property "Reference" "R11"
+		(property "Reference" "R114"
 			(at 124.46 70.358 90)
 			(show_name no)
@@
 			(project "gatebench"
 				(path "/f24451ff-caac-4926-9774-6edc1451b63f/a3c4557c-c544-4f42-ade0-8584472233ea"
-					(reference "R11")
+					(reference "R114")
 					(unit 1)
 				)
@@
 		(in_pos_files yes)
 		(dnp no)
-		(property "Reference" "R23"
+		(property "Reference" "R123"
 			(at 179.07 93.218 90)
 			(show_name no)
@@
 			(project "gatebench"
 				(path "/f24451ff-caac-4926-9774-6edc1451b63f/a3c4557c-c544-4f42-ade0-8584472233ea"
-					(reference "R23")
+					(reference "R123")
 					(unit 1)
 				)
@@
 		(in_pos_files yes)
 		(dnp no)
-		(property "Reference" "TP34"
+		(property "Reference" "TP38"
 			(at 214.122 59.69 90)
 			(show_name no)
@@
 			(project "gatebench"
 				(path "/f24451ff-caac-4926-9774-6edc1451b63f/a3c4557c-c544-4f42-ade0-8584472233ea"
-					(reference "TP34")
+					(reference "TP38")
 					(unit 1)
 				)
@@
 		(in_pos_files yes)
 		(dnp no)
-		(property "Reference" "R22"
+		(property "Reference" "R122"
 			(at 166.116 108.458 90)
 			(show_name no)
@@
 			(project "gatebench"
 				(path "/f24451ff-caac-4926-9774-6edc1451b63f/a3c4557c-c544-4f42-ade0-8584472233ea"
-					(reference "R22")
+					(reference "R122")
 					(unit 1)
 				)
@@
 		(in_pos_files yes)
 		(dnp no)
-		(property "Reference" "R17"
+		(property "Reference" "R120"
 			(at 124.46 105.918 90)
 			(show_name no)
@@
 			(project "gatebench"
 				(path "/f24451ff-caac-4926-9774-6edc1451b63f/a3c4557c-c544-4f42-ade0-8584472233ea"
-					(reference "R17")
+					(reference "R120")
 					(unit 1)
 				)
@@
 		(in_pos_files yes)
 		(dnp no)
-		(property "Reference" "R18"
+		(property "Reference" "R121"
 			(at 124.46 110.998 90)
 			(show_name no)
@@
 			(project "gatebench"
 				(path "/f24451ff-caac-4926-9774-6edc1451b63f/a3c4557c-c544-4f42-ade0-8584472233ea"
-					(reference "R18")
+					(reference "R121")
 					(unit 1)
 				)
@@
 		(in_pos_files yes)
 		(dnp no)
-		(property "Reference" "R14"
+		(property "Reference" "R117"
 			(at 124.46 88.138 90)
 			(show_name no)
@@
 			(project "gatebench"
 				(path "/f24451ff-caac-4926-9774-6edc1451b63f/a3c4557c-c544-4f42-ade0-8584472233ea"
-					(reference "R14")
+					(reference "R117")
 					(unit 1)
 				)
@@
 		(in_pos_files yes)
 		(dnp no)
-		(property "Reference" "R10"
+		(property "Reference" "R113"
 			(at 124.46 65.278 90)
 			(show_name no)
@@
 			(project "gatebench"
 				(path "/f24451ff-caac-4926-9774-6edc1451b63f/a3c4557c-c544-4f42-ade0-8584472233ea"
-					(reference "R10")
+					(reference "R113")
 					(unit 1)
 				)
@@
 		(in_pos_files yes)
 		(dnp no)
-		(property "Reference" "R24"
+		(property "Reference" "R124"
 			(at 179.07 98.298 90)
 			(show_name no)
@@
 			(project "gatebench"
 				(path "/f24451ff-caac-4926-9774-6edc1451b63f/a3c4557c-c544-4f42-ade0-8584472233ea"
-					(reference "R24")
+					(reference "R124")
 					(unit 1)
 				)
@@
 		(in_pos_files yes)
 		(dnp no)
-		(property "Reference" "TP33"
+		(property "Reference" "TP39"
 			(at 214.122 64.77 90)
 			(show_name no)
@@
 			(project "gatebench"
 				(path "/f24451ff-caac-4926-9774-6edc1451b63f/a3c4557c-c544-4f42-ade0-8584472233ea"
-					(reference "TP33")
+					(reference "TP39")
 					(unit 1)
 				)
@@
 		(dnp no)
 		(fields_autoplaced yes)
-		(property "Reference" "#PWR057"
+		(property "Reference" "#PWR0176"
 			(at 148.59 111.76 0)
 			(hide yes)
@@
 			(project "gatebench"
 				(path "/f24451ff-caac-4926-9774-6edc1451b63f/a3c4557c-c544-4f42-ade0-8584472233ea"
-					(reference "#PWR057")
+					(reference "#PWR0176")
 					(unit 1)
 				)
@@
 		(in_pos_files yes)
 		(dnp no)
-		(property "Reference" "R16"
+		(property "Reference" "R119"
 			(at 124.46 100.838 90)
 			(show_name no)
@@
 			(project "gatebench"
 				(path "/f24451ff-caac-4926-9774-6edc1451b63f/a3c4557c-c544-4f42-ade0-8584472233ea"
-					(reference "R16")
+					(reference "R119")
 					(unit 1)
 				)
@@
 		(in_pos_files yes)
 		(dnp no)
-		(property "Reference" "TP37"
+		(property "Reference" "TP35"
 			(at 214.122 44.45 90)
 			(show_name no)
@@
 			(project "gatebench"
 				(path "/f24451ff-caac-4926-9774-6edc1451b63f/a3c4557c-c544-4f42-ade0-8584472233ea"
-					(reference "TP37")
+					(reference "TP35")
 					(unit 1)
 				)
@@
 		(in_pos_files yes)
 		(dnp no)
-		(property "Reference" "R13"
+		(property "Reference" "R116"
 			(at 124.46 83.058 90)
 			(show_name no)
@@
 			(project "gatebench"
 				(path "/f24451ff-caac-4926-9774-6edc1451b63f/a3c4557c-c544-4f42-ade0-8584472233ea"
-					(reference "R13")
-					(unit 1)
-				)
+					(reference "R116")
+					(unit 1)
+				)
