File: hardware/ws2812b.kicad_sch (KiCad schematic)
At the start: 28 parts, among them U6 74AHCT1G125

Commit message: feat(hw): closing sch, starting pcb
Parts:
- renumbered C12 to C25, C32 to C26, C15 to C27, C31 to C28, C23 to C29, C24 to C31, C29 to C32, C25 to C33, C28 to C34, C26 to C35, C27 to C36, D14 to D10, D6 to D11, D13 to D12, D7 to D13, D12 to D14, D8 to D15, D11 to D16, D9 to D17, D10 to D18, D5 to D9, R29 to R125, TP49 to TP40, TP50 to TP41, TP52 to TP42, TP51 to TP43, U6 to U9
